Commit message: Update _local.urdf mesh path

File: mycobot_description/urdf/mycobot/mycobot_with_gripper_parallel_local.urdf (robot description, URDF)
Before this commit: robot mycobot_280pi, 17 links, 16 joints
Links:
- link base_mount: geometry collision mesh filename=../../meshes/arm/base_mount.dae; visual mesh filename=../../meshes/arm/base_mount.dae
- link gripper_base: geometry collision mesh filename=../../meshes/gripper/gripper_base.dae; visual mesh filename=../../meshes/gripper/gripper_base.dae
- link left_finger: geometry collision mesh filename=../../meshes/gripper/left_finger.dae; visual mesh filename=../../meshes/gripper/left_finger.dae
- link left_inner_knuckle: geometry collision mesh filename=../../meshes/gripper/left_inner_knuckle.dae; visual mesh filename=../../meshes/gripper/left_inner_knuckle.dae
- link left_outer_knuckle: geometry collision mesh filename=../../meshes/gripper/left_outer_knuckle.dae; visual mesh filename=../../meshes/gripper/left_outer_knuckle.dae
- link link1: geometry collision mesh filename=../../meshes/arm/link1.dae; visual mesh filename=../../meshes/arm/link1.dae
- link link2: geometry collision mesh filename=../../meshes/arm/link2.dae; visual mesh filename=../../meshes/arm/link2.dae
- link link3: geometry collision mesh filename=../../meshes/arm/link3.dae; visual mesh filename=../../meshes/arm/link3.dae
- link link4: geometry collision mesh filename=../../meshes/arm/link4.dae; visual mesh filename=../../meshes/arm/link4.dae
- link link5: geometry collision mesh filename=../../meshes/arm/link5.dae; visual mesh filename=../../meshes/arm/link5.dae
- link link6: geometry collision mesh filename=../../meshes/arm/link6.dae; visual mesh filename=../../meshes/arm/link6.dae
- link link_base: geometry collision mesh filename=../../meshes/arm/link_base.dae; visual mesh filename=../../meshes/arm/link_base.dae
- link right_finger: geometry collision mesh filename=../../meshes/gripper/right_finger.dae; visual mesh filename=../../meshes/gripper/right_finger.dae
- link right_inner_knuckle: geometry collision mesh filename=../../meshes/gripper/right_inner_knuckle.dae; visual mesh filename=../../meshes/gripper/right_inner_knuckle.dae
- link right_outer_knuckle: geometry collision mesh filename=../../meshes/gripper/right_outer_knuckle.dae; visual mesh filename=../../meshes/gripper/right_outer_knuckle.dae
